File: PicoDVI-N64_PCB/PicoDVI-N64.kicad_pcb (KiCad board)
At the start: 2 copper layers, 53.9 x 37.9 mm, 14 parts, among them J4 NOT_HDMI_A, X1 3-1734592-0

Commit message: Add files via upload
Other:
- board size 53.9 x 37.9 mm -> 53.3 x 36.3 mm
